File: hardware/open-lego-camera-cm4.kicad_sch (KiCad schematic)
At the start: 45 parts, among them J1 USB-C Charge/Data, J2 LiPo 1S, J3 microSD, J4 CSI Camera 0, J5 CSI Camera 1, J6 DSI LCD Display, J7 Speaker, J8 IO Header, U1 MCP73871, U2 MAX17048, U3 TPS63020 -> +5V, U4 AP2112K -> +3V3, U5 Raspberry Pi CM4, U6 ICS-43434 (L), U7 ICS-43434 (R), U8 MAX98357A

Commit message: Add footprints and complete all component connections
Assign a standard KiCad footprint to every component and wire up all
previously optional/dangling pins so no functional pin floats.

Footprints: every symbol now maps to a KiCad 7/8 library footprint
(0603 passives, QFN/SOT/TDFN/VSON ICs, USB-C, JST-PH, microSD, 15-pin
FFC, pin headers, LEDs, test points).

Connections completed:
- USB-C D+/D- routed to the CM4 USB pins
- Charger CE tied high / TE low; PROG1/PROG2 current-set resistors;
  STAT1/STAT2/PG drive status LEDs D1-D3
- Fuel gauge QSTRT tied low; FUEL_ALRT to CM4 GPIO24
- Camera enable/LED lines to CM4 GPIO4/27 and GPIO22/23
- MAX98357A GAIN set (100k to GND); SD_MODE pull-up
- GLOBAL_EN/nRPIBOOT pull-ups plus a boot-mode jumper (J9) on nRPIBOOT
- Test points TP1-TP3 for CM4 +3V3 out, RUN_PG and SD_VDD_EN
- Decoupling on the CM4 3V3 output

ERC now shows no single-endpoint nets. README updated with the wiring
summary, footprint notes, and new BOM entries.

Co-Authored-By: Claude Opus 4.8 <noreply@anthropic.com>
Claude-Session: https://claude.ai/code/session_01595tDoeEay2LaGDFsf3aE5
Parts:
- added C11: 4.7uF, Capacitor_SMD:C_0603_1608Metric, symbol olc:C
- added D1: CHG, LED_SMD:LED_0603_1608Metric, symbol olc:LED
- added D2: STDBY, LED_SMD:LED_0603_1608Metric, symbol olc:LED
- added D3: PWR, LED_SMD:LED_0603_1608Metric, symbol olc:LED
- added J9: BOOT jumper, Connector_PinHeader_2.54mm:PinHeader_1x02_P2.54mm_Vertical, symbol olc:Conn_2pin
- added R19, R20, R21: 1k, Resistor_SMD:R_0603_1608Metric, symbol olc:R
- added R22: 100k GAIN, Resistor_SMD:R_0603_1608Metric, symbol olc:R
- added R23: 1.2k PROG2, Resistor_SMD:R_0603_1608Metric, symbol olc:R
- added TP1: 3V3_CM4, TestPoint:TestPoint_Pad_D1.5mm, symbol olc:TestPoint
- added TP2: RUN_PG, TestPoint:TestPoint_Pad_D1.5mm, symbol olc:TestPoint
- added TP3: SD_VDD_EN, TestPoint:TestPoint_Pad_D1.5mm, symbol olc:TestPoint
- C1, C10, C2, C3, C4, C5, C6, C7, C8, C9: footprint (none) -> Capacitor_SMD:C_0603_1608Metric
- J1: footprint (none) -> Connector_USB:USB_C_Receptacle_GCT_USB4085
- J2, J7: footprint (none) -> Connector_JST:JST_PH_B2B-PH-K_1x02_P2.00mm_Vertical
- J3: footprint (none) -> Connector_Card:microSD_HC_Hirose_DM3AT-SF-PEJM5
- J4, J5, J6: footprint (none) -> Connector_FFC-FPC:Hirose_FH12-15S-1SH_1x15-1MP_P1.00mm_Horizontal
- J8: footprint (none) -> Connector_PinHeader_2.54mm:PinHeader_2x05_P2.54mm_Vertical
- L1: footprint (none) -> Inductor_SMD:L_Bourns-SRN6045TA_6.0x6.0mm
- R1, R10, R11, R12, R13, R14, R15, R16, R17, R18, R2, R4, R5, R6, R7, R8, R9: footprint (none) -> Resistor_SMD:R_0603_1608Metric
- R3: value 2k PROG -> 2k PROG1; footprint (none) -> Resistor_SMD:R_0603_1608Metric
- U1: footprint (none) -> Package_DFN_QFN:QFN-20-1EP_4x4mm_P0.5mm_EP2.6x2.6mm
- U2: footprint (none) -> Package_DFN_QFN:TDFN-8-1EP_2x3mm_P0.5mm_EP0.9x1.5mm
- U3: footprint (none) -> Package_DFN_QFN:VSON-14_3x4mm_P0.5mm
- U4: footprint (none) -> Package_TO_SOT_SMD:SOT-23-5
- U5: footprint (none) -> Connector_Hirose:Hirose_DF40C-100DS-0.4V_2x50-1MP_P0.40mm_Vertical
- U6, U7: footprint (none) -> Sensor_Audio:Knowles_LGA-6_3.5x2.65mm
- U8: footprint (none) -> Package_DFN_QFN:QFN-16-1EP_3x3mm_P0.5mm_EP1.75x1.75mm
Connections:
- net +3V3: now also R19.1, R20.1, R21.1
- net +3V3_CM4: now also C11.1, TP1.1
- net AMP_GAIN: now also R22.1
- net CAM0_GPIO: now also U5.G4 (GPIO4_CAM0_EN)
- net CAM0_LED: now also U5.G22 (GPIO22_CAM0_LED)
- net CAM1_GPIO: now also U5.G27 (GPIO27_CAM1_EN)
- net CAM1_LED: now also U5.G23 (GPIO23_CAM1_LED)
- net CHG_PG: now also D3.2 (K)
- net CHG_PROG2: now also R23.1
- net CHG_STAT1: now also D1.2 (K)
- net CHG_STAT2: now also D2.2 (K)
- net FUEL_ALRT: now also U5.G24 (GPIO24_FUEL_ALRT)
- net GND: now also U1.14 (TE), U2.7 (QSTRT), C11.2, J9.2, R22.2, R23.2; no longer U1.13 (CE)
- net RUN_PG: now also TP2.1
- net SD_VDD_EN: now also TP3.1
- net USB_DN: now also U5.UDN (USB_DN)
- net USB_DP: now also U5.UDP (USB_DP)
- net VBUS_USB: now also U1.13 (CE)
- net VSYS: no longer U1.14 (TE)
- net nRPIBOOT: now also J9.1
- new net PG_A: D3.1 (A), R21.2
- new net STAT1_A: D1.1 (A), R19.2
- new net STAT2_A: D2.1 (A), R20.2

Commit message: Fix PCB footprint assignments so Update-PCB-from-Schematic is clean
Update PCB from Schematic reported 11 footprints not found because some
library names were guessed. Correct them against the official KiCad
footprint repository:
- ICS-43434 mics -> Sensor_Audio:InvenSense_ICS-43434-6_3.5x2.65mm
- MAX17048      -> Package_DFN_QFN:DFN-8-1EP_2x3mm_P0.5mm_EP0.61x2.2mm
- TPS63020      -> Package_DFN_QFN:DFN-14-1EP_3x4mm_P0.5mm_EP1.7x3.3mm
- CSI/DSI FFC   -> Connector_FFC-FPC:Molex_200528-0150_1x15-1MP_P1.00mm_Horizontal
- Inductor L1   -> Inductor_SMD:L_Bourns_SRN6045TA

Stock KiCad has no CM4/DF40-100 footprint, and the functional CM4 symbol's
pin numbers won't map to any generic connector. Add a local placeholder
footprint (open-lego-camera.pretty/CM4_Functional.kicad_mod) whose 54 pads
are named to match the symbol pins exactly, plus an fp-lib-table to
register the library, so every CM4 net maps and the board is fully
routable. The placeholder must still be replaced with the real dual DF40
connectors before fabrication.

FLG2/FLG3 have no footprint by design (power flags) and are correctly
skipped. README updated.

Co-Authored-By: Claude Opus 4.8 <noreply@anthropic.com>
Claude-Session: https://claude.ai/code/session_01595tDoeEay2LaGDFsf3aE5
Parts:
- J4, J5, J6: footprint Connector_FFC-FPC:Hirose_FH12-15S-1SH_1x15-1MP_P1.00mm_Horizontal -> Connector_FFC-FPC:Molex_200528-0150_1x15-1MP_P1.00mm_Horizontal
- L1: footprint Inductor_SMD:L_Bourns-SRN6045TA_6.0x6.0mm -> Inductor_SMD:L_Bourns_SRN6045TA
- U2: footprint Package_DFN_QFN:TDFN-8-1EP_2x3mm_P0.5mm_EP0.9x1.5mm -> Package_DFN_QFN:DFN-8-1EP_2x3mm_P0.5mm_EP0.61x2.2mm
- U3: footprint Package_DFN_QFN:VSON-14_3x4mm_P0.5mm -> Package_DFN_QFN:DFN-14-1EP_3x4mm_P0.5mm_EP1.7x3.3mm
- U5: footprint Connector_Hirose:Hirose_DF40C-100DS-0.4V_2x50-1MP_P0.40mm_Vertical -> open-lego-camera:CM4_Functional
- U6, U7: footprint Sensor_Audio:Knowles_LGA-6_3.5x2.65mm -> Sensor_Audio:InvenSense_ICS-43434-6_3.5x2.65mm
Changed lines of the file:
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@@
     (property "Value" "MAX17048" (at 200.00 240.16 0)
       (effects (font (size 1.27 1.27))))
-    (property "Footprint" "Package_DFN_QFN:TDFN-8-1EP_2x3mm_P0.5mm_EP0.9x1.5mm" (at 200.00 230.00 0)
+    (property "Footprint" "Package_DFN_QFN:DFN-8-1EP_2x3mm_P0.5mm_EP0.61x2.2mm" (at 200.00 230.00 0)
       (effects (font (size 1.27 1.27)) hide))
     (property "Datasheet" "~" (at 200.00 230.00 0)
@@
     (property "Value" "TPS63020 -> +5V" (at 200.00 331.43 0)
       (effects (font (size 1.27 1.27))))
-    (property "Footprint" "Package_DFN_QFN:VSON-14_3x4mm_P0.5mm" (at 200.00 320.00 0)
+    (property "Footprint" "Package_DFN_QFN:DFN-14-1EP_3x4mm_P0.5mm_EP1.7x3.3mm" (at 200.00 320.00 0)
       (effects (font (size 1.27 1.27)) hide))
     (property "Datasheet" "~" (at 200.00 320.00 0)
@@
     (property "Value" "1.5uH" (at 260.00 307.62 0)
       (effects (font (size 1.27 1.27))))
-    (property "Footprint" "Inductor_SMD:L_Bourns-SRN6045TA_6.0x6.0mm" (at 260.00 300.00 0)
+    (property "Footprint" "Inductor_SMD:L_Bourns_SRN6045TA" (at 260.00 300.00 0)
       (effects (font (size 1.27 1.27)) hide))
     (property "Datasheet" "~" (at 260.00 300.00 0)
@@
     (property "Value" "Raspberry Pi CM4" (at 480.00 233.18 0)
       (effects (font (size 1.27 1.27))))
-    (property "Footprint" "Connector_Hirose:Hirose_DF40C-100DS-0.4V_2x50-1MP_P0.40mm_Vertical" (at 480.00 190.00 0)
+    (property "Footprint" "open-lego-camera:CM4_Functional" (at 480.00 190.00 0)
       (effects (font (size 1.27 1.27)) hide))
     (property "Datasheet" "~" (at 480.00 190.00 0)
@@
     (property "Value" "CSI Camera 0" (at 780.00 125.24 0)
       (effects (font (size 1.27 1.27))))
-    (property "Footprint" "Connector_FFC-FPC:Hirose_FH12-15S-1SH_1x15-1MP_P1.00mm_Horizontal" (at 780.00 110.00 0)
+    (property "Footprint" "Connector_FFC-FPC:Molex_200528-0150_1x15-1MP_P1.00mm_Horizontal" (at 780.00 110.00 0)
       (effects (font (size 1.27 1.27)) hide))
     (property "Datasheet" "~" (at 780.00 110.00 0)
@@
     (property "Value" "CSI Camera 1" (at 780.00 215.24 0)
       (effects (font (size 1.27 1.27))))
-    (property "Footprint" "Connector_FFC-FPC:Hirose_FH12-15S-1SH_1x15-1MP_P1.00mm_Horizontal" (at 780.00 200.00 0)
+    (property "Footprint" "Connector_FFC-FPC:Molex_200528-0150_1x15-1MP_P1.00mm_Horizontal" (at 780.00 200.00 0)
       (effects (font (size 1.27 1.27)) hide))
     (property "Datasheet" "~" (at 780.00 200.00 0)
@@
     (property "Value" "DSI LCD Display" (at 780.00 305.24 0)
       (effects (font (size 1.27 1.27))))
-    (property "Footprint" "Connector_FFC-FPC:Hirose_FH12-15S-1SH_1x15-1MP_P1.00mm_Horizontal" (at 780.00 290.00 0)
+    (property "Footprint" "Connector_FFC-FPC:Molex_200528-0150_1x15-1MP_P1.00mm_Horizontal" (at 780.00 290.00 0)
       (effects (font (size 1.27 1.27)) hide))
     (property "Datasheet" "~" (at 780.00 290.00 0)
@@
     (property "Value" "ICS-43434 (L)" (at 780.00 360.16 0)
       (effects (font (size 1.27 1.27))))
-    (property "Footprint" "Sensor_Audio:Knowles_LGA-6_3.5x2.65mm" (at 780.00 350.00 0)
+    (property "Footprint" "Sensor_Audio:InvenSense_ICS-43434-6_3.5x2.65mm" (at 780.00 350.00 0)
       (effects (font (size 1.27 1.27)) hide))
     (property "Datasheet" "~" (at 780.00 350.00 0)
@@
     (property "Value" "ICS-43434 (R)" (at 780.00 430.16 0)
       (effects (font (size 1.27 1.27))))
-    (property "Footprint" "Sensor_Audio:Knowles_LGA-6_3.5x2.65mm" (at 780.00 420.00 0)
+    (property "Footprint" "Sensor_Audio:InvenSense_ICS-43434-6_3.5x2.65mm" (at 780.00 420.00 0)
       (effects (font (size 1.27 1.27)) hide))
     (property "Datasheet" "~" (at 780.00 420.00 0)
