File: hardware/cm4-carrier/cm4.kicad_sch (KiCad schematic)
At the start: 4 parts, among them J3 Raspberry Pi CM4, J4 Raspberry Pi CM4

Commit message: Add stereo I2S audio (2x ICS-43434 mics + 2x MAX98357A amps)
Add an audio.kicad_sch sub-sheet with stereo microphone capture and stereo
speaker output over the CM4's I2S peripheral:

- 2x ICS-43434 I2S MEMS mics (U8 Left = LR->GND, U9 Right = LR->VDD) sharing
  the I2S RX bus, powered at 3.3V, with decoupling.
- 2x MAX98357A I2S class-D amps (U10 Left, U11 Right) on the I2S TX bus,
  powered at 5V; channel selected by the SD_MODE resistor divider, GAIN_SLOT
  set via 100k, VDD bulk/decoupling. Filterless BTL outputs go straight to the
  speaker connector.
- 4-pin 1.25mm (JST GH) speaker connector J9 = SPK_L+/L-/R+/R-.

The CM4 sheet exports the I2S bus (GPIO18=BCLK, GPIO19=LRCLK, GPIO20=PCM_DIN,
GPIO21=PCM_DOUT) as global nets I2S_CLK/FS/DIN/DOUT; the audio sheet consumes
them. Both mics+amps share BCLK/LRCLK; mics drive DIN, amps receive DOUT.

Pinouts: ICS-43434 from KiCad Sensor_Audio; MAX98357A (TQFN-16) from KiCad
symbol MR !3846; JST GH 4-pin footprint from KiCad. Root gains a (pinless)
Stereo Audio box (page 9, now 8 sub-sheets). README/BOM updated. No format
change (KiCad 10, 20260306).

Co-Authored-By: Claude Opus 4.8 <noreply@anthropic.com>
Claude-Session: https://claude.ai/code/session_015B7X7FE461jFSRaiTFdnFt
Connections:
- net I2S_DOUT: now reaches J3.25 (GPIO21)
- net I2S_FS: now reaches J3.26 (GPIO19)
- net I2S_DIN: now reaches J3.27 (GPIO20)
- net I2S_CLK: now reaches J3.49 (GPIO18)
