File: hardware/cm4-carrier/regulator.kicad_sch (KiCad schematic)
At the start: 9 parts, among them U2 TPS61088

Commit message: Add Dynamic Power Path Management and battery protection
Rework the power architecture to add DPPM and dedicated cell protection.

Power path (DPPM): replace the MCP73831 with a TI BQ24075 USB-friendly
charger whose OUT pin is a separate system rail (SYS). The load now runs
directly from USB when present (system works with a dead/absent battery and
the cell is not needlessly cycled) and falls back to the battery when USB is
removed, while the cell charges from the remaining input budget. Adds ISET,
ILIM and TMR programming resistors, EN1/EN2/CE/SYSOFF strapping, a 10k NTC
on TS for battery-temperature protection, and CHG/PGOOD status LEDs. The
5 V boost regulator now draws from SYS instead of VBAT.

Battery protection: new battery_protection.kicad_sch sub-sheet with an
AP9101CK6 1-cell protection controller (DW01A-class) driving an FS8205A dual
N-MOSFET in the cell's negative line — over-charge, over-discharge,
over-current and short-circuit cutoff. The raw JST cell connector moves here;
its protected terminals feed VBAT/GND to the rest of the board.

Pinouts for BQ24075 and AP9101CK6 were taken from KiCad's Battery_Management
library. Root sheet gains the Battery Protection box and the SYS net; all
hierarchical labels match their sheet pins and reference designators are
globally unique. README/BOM updated. No format change (KiCad 10, 20260306).

Co-Authored-By: Claude Opus 4.8 <noreply@anthropic.com>
Claude-Session: https://claude.ai/code/session_015B7X7FE461jFSRaiTFdnFt
Connections:
- net VBAT renamed SYS
Other:
- note added: "5 V boost regulator (TPS61088) - SYS (3.0-4.4V) -> 5V/3A"
- note removed: "5 V boost regulator (TPS61088, LiPo 3.0-4.2V -> 5V/3A)"
Changed lines of the file:
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@@
 	(generator_version "10.0")
 	(paper "A3")
-	(text "5 V boost regulator (TPS61088, LiPo 3.0-4.2V -> 5V/3A)" (at 20.00 12.00 0)
+	(text "5 V boost regulator (TPS61088) - SYS (3.0-4.4V) -> 5V/3A" (at 20.00 12.00 0)
 		(effects (font (size 2.0 2.0)) (justify left))
 )
@@
 		(instances
 			(project "cm4-carrier"
-				(path "/a2053281-5c44-4a85-a311-f1d495df0c08/649d7749-8e9e-4a0b-bbc9-e348fe913b1e"
+				(path "/de8be509-02ff-4a5f-a12c-6d0038f6bb72/3b86b796-8442-443c-8844-40de3caddd6a"
 					(reference "U2") (unit 1))))
 	)
-	(hierarchical_label "VBAT" (shape input) (at 30.00 40.00 180)
+	(hierarchical_label "SYS" (shape input) (at 30.00 40.00 180)
 		(effects (font (size 1.27 1.27)) (justify left))
 )
@@
 		(stroke (width 0) (type default))
 	)
-	(label "VBAT" (at 40.00 40.00 0)
+	(label "SYS" (at 40.00 40.00 0)
 		(effects (font (size 1.27 1.27)) (justify left bottom))
 )
@@
 		(stroke (width 0) (type default))
 	)
-	(label "VBAT" (at 74.76 48.65 180)
+	(label "SYS" (at 74.76 48.65 180)
 		(effects (font (size 1.27 1.27)) (justify right bottom))
 )
@@
 		(stroke (width 0) (type default))
 	)
-	(label "VBAT" (at 74.76 51.19 180)
+	(label "SYS" (at 74.76 51.19 180)
 		(effects (font (size 1.27 1.27)) (justify right bottom))
 )
@@
 		(instances
 			(project "cm4-carrier"
-				(path "/a2053281-5c44-4a85-a311-f1d495df0c08/649d7749-8e9e-4a0b-bbc9-e348fe913b1e"
+				(path "/de8be509-02ff-4a5f-a12c-6d0038f6bb72/3b86b796-8442-443c-8844-40de3caddd6a"
 					(reference "#PWR001") (unit 1))))
 	)
@@
 		(instances
 			(project "cm4-carrier"
-				(path "/a2053281-5c44-4a85-a311-f1d495df0c08/649d7749-8e9e-4a0b-bbc9-e348fe913b1e"
+				(path "/de8be509-02ff-4a5f-a12c-6d0038f6bb72/3b86b796-8442-443c-8844-40de3caddd6a"
 					(reference "#PWR002") (unit 1))))
 	)
@@
 		(instances
 			(project "cm4-carrier"
-				(path "/a2053281-5c44-4a85-a311-f1d495df0c08/649d7749-8e9e-4a0b-bbc9-e348fe913b1e"
+				(path "/de8be509-02ff-4a5f-a12c-6d0038f6bb72/3b86b796-8442-443c-8844-40de3caddd6a"
 					(reference "#PWR003") (unit 1))))
 	)
@@
 		(instances
 			(project "cm4-carrier"
-				(path "/a2053281-5c44-4a85-a311-f1d495df0c08/649d7749-8e9e-4a0b-bbc9-e348fe913b1e"
+				(path "/de8be509-02ff-4a5f-a12c-6d0038f6bb72/3b86b796-8442-443c-8844-40de3caddd6a"
 					(reference "L1") (unit 1))))
 	)
@@
 		(stroke (width 0) (type default))
 	)
-	(label "VBAT" (at 81.11 95.00 180)
+	(label "SYS" (at 81.11 95.00 180)
 		(effects (font (size 1.27 1.27)) (justify right bottom))
 )
@@
 		(instances
 			(project "cm4-carrier"
-				(path "/a2053281-5c44-4a85-a311-f1d495df0c08/649d7749-8e9e-4a0b-bbc9-e348fe913b1e"
+				(path "/de8be509-02ff-4a5f-a12c-6d0038f6bb72/3b86b796-8442-443c-8844-40de3caddd6a"
 					(reference "R5") (unit 1))))
 	)
@@
 		(instances
 			(project "cm4-carrier"
-				(path "/a2053281-5c44-4a85-a311-f1d495df0c08/649d7749-8e9e-4a0b-bbc9-e348fe913b1e"
+				(path "/de8be509-02ff-4a5f-a12c-6d0038f6bb72/3b86b796-8442-443c-8844-40de3caddd6a"
 					(reference "R6") (unit 1))))
 	)
@@
 		(instances
 			(project "cm4-carrier"
-				(path "/a2053281-5c44-4a85-a311-f1d495df0c08/649d7749-8e9e-4a0b-bbc9-e348fe913b1e"
+				(path "/de8be509-02ff-4a5f-a12c-6d0038f6bb72/3b86b796-8442-443c-8844-40de3caddd6a"
 					(reference "#PWR004") (unit 1))))
 	)
@@
 		(instances
 			(project "cm4-carrier"
-				(path "/a2053281-5c44-4a85-a311-f1d495df0c08/649d7749-8e9e-4a0b-bbc9-e348fe913b1e"
+				(path "/de8be509-02ff-4a5f-a12c-6d0038f6bb72/3b86b796-8442-443c-8844-40de3caddd6a"
 					(reference "C5") (unit 1))))
 	)
@@
 		(instances
 			(project "cm4-carrier"
-				(path "/a2053281-5c44-4a85-a311-f1d495df0c08/649d7749-8e9e-4a0b-bbc9-e348fe913b1e"
+				(path "/de8be509-02ff-4a5f-a12c-6d0038f6bb72/3b86b796-8442-443c-8844-40de3caddd6a"
 					(reference "#PWR005") (unit 1))))
 	)
@@
 		(instances
 			(project "cm4-carrier"
-				(path "/a2053281-5c44-4a85-a311-f1d495df0c08/649d7749-8e9e-4a0b-bbc9-e348fe913b1e"
+				(path "/de8be509-02ff-4a5f-a12c-6d0038f6bb72/3b86b796-8442-443c-8844-40de3caddd6a"
 					(reference "C6") (unit 1))))
 	)
@@
 		(instances
 			(project "cm4-carrier"
-				(path "/a2053281-5c44-4a85-a311-f1d495df0c08/649d7749-8e9e-4a0b-bbc9-e348fe913b1e"
+				(path "/de8be509-02ff-4a5f-a12c-6d0038f6bb72/3b86b796-8442-443c-8844-40de3caddd6a"
 					(reference "#PWR006") (unit 1))))
 	)
@@
 		(instances
 			(project "cm4-carrier"
-				(path "/a2053281-5c44-4a85-a311-f1d495df0c08/649d7749-8e9e-4a0b-bbc9-e348fe913b1e"
+				(path "/de8be509-02ff-4a5f-a12c-6d0038f6bb72/3b86b796-8442-443c-8844-40de3caddd6a"
 					(reference "C3") (unit 1))))
 	)
@@
 		(stroke (width 0) (type default))
 	)
-	(label "VBAT" (at 36.19 54.92 90)
+	(label "SYS" (at 36.19 54.92 90)
 		(effects (font (size 1.27 1.27)) (justify left bottom))
 )
@@
 		(instances
 			(project "cm4-carrier"
-				(path "/a2053281-5c44-4a85-a311-f1d495df0c08/649d7749-8e9e-4a0b-bbc9-e348fe913b1e"
+				(path "/de8be509-02ff-4a5f-a12c-6d0038f6bb72/3b86b796-8442-443c-8844-40de3caddd6a"
 					(reference "#PWR007") (unit 1))))
 	)
@@
 		(instances
 			(project "cm4-carrier"
-				(path "/a2053281-5c44-4a85-a311-f1d495df0c08/649d7749-8e9e-4a0b-bbc9-e348fe913b1e"
+				(path "/de8be509-02ff-4a5f-a12c-6d0038f6bb72/3b86b796-8442-443c-8844-40de3caddd6a"
 					(reference "C4") (unit 1))))
 	)
@@
 		(instances
 			(project "cm4-carrier"
-				(path "/a2053281-5c44-4a85-a311-f1d495df0c08/649d7749-8e9e-4a0b-bbc9-e348fe913b1e"
+				(path "/de8be509-02ff-4a5f-a12c-6d0038f6bb72/3b86b796-8442-443c-8844-40de3caddd6a"
 					(reference "#PWR008") (unit 1))))
 	)
@@
 		(instances
 			(project "cm4-carrier"
-				(path "/a2053281-5c44-4a85-a311-f1d495df0c08/649d7749-8e9e-4a0b-bbc9-e348fe913b1e"
+				(path "/de8be509-02ff-4a5f-a12c-6d0038f6bb72/3b86b796-8442-443c-8844-40de3caddd6a"
 					(reference "C7") (unit 1))))
 	)
@@
 		(instances
 			(project "cm4-carrier"
-				(path "/a2053281-5c44-4a85-a311-f1d495df0c08/649d7749-8e9e-4a0b-bbc9-e348fe913b1e"
+				(path "/de8be509-02ff-4a5f-a12c-6d0038f6bb72/3b86b796-8442-443c-8844-40de3caddd6a"
 					(reference "#PWR009") (unit 1))))
 	)
