File: hardware/cm4-carrier/battery_monitor.kicad_sch (KiCad schematic)
At the start: 5 parts, among them U3 MAX17048G+T

Commit message: Fix four footprint identifiers not found in KiCad libraries
"Update PCB from Schematic" reported four footprints missing; correct them to
the actual names in the current KiCad libraries (edited in place to preserve
symbol UUIDs, so existing PCB associations are kept):

- J1 USB-C: USB_C_Receptacle_GCT_USB4110-GF-A_16P_TopMnt_Horizontal
            -> USB_C_Receptacle_GCT_USB4110
- L1 inductor: L_Bourns-SRP1265A -> L_Bourns_SRP1245A (SRP1265A not in KiCad;
  pick the footprint matching your actual boost inductor)
- U1 BQ24075: VQFN-16-1EP_3x3mm_P0.5mm_EP1.7x1.7mm
            -> QFN-16-1EP_3x3mm_P0.5mm_EP1.7x1.7mm
- U3 MAX17048: DFN-8-1EP_2x2mm_P0.5mm_EP0.61x1.42mm
            -> DFN-8-1EP_2x2mm_P0.5mm_EP0.9x1.5mm

README BOM updated to match.

Co-Authored-By: Claude Opus 4.8 <noreply@anthropic.com>
Claude-Session: https://claude.ai/code/session_015B7X7FE461jFSRaiTFdnFt
Parts:
- U3: footprint Package_DFN_QFN:DFN-8-1EP_2x2mm_P0.5mm_EP0.61x1.42mm -> Package_DFN_QFN:DFN-8-1EP_2x2mm_P0.5mm_EP0.9x1.5mm
Changed lines of the file:
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@@
 		(property "Value" "MAX17048G+T" (at 90.00 63.89 0)
 			(effects (font (size 1.27 1.27)) (justify left)))
-		(property "Footprint" "Package_DFN_QFN:DFN-8-1EP_2x2mm_P0.5mm_EP0.61x1.42mm" (at 90.00 55.00 90)
+		(property "Footprint" "Package_DFN_QFN:DFN-8-1EP_2x2mm_P0.5mm_EP0.9x1.5mm" (at 90.00 55.00 90)
 			(effects (font (size 1.27 1.27)) (hide yes)))
 		(property "Datasheet" "https://www.analog.com/media/en/technical-documentation/data-sheets/MAX17048-MAX17049.pdf" (at 90.00 55.00 0)

Commit message: hardware: fix J1/U3 symbol pad mapping for PCB update
Two custom symbols used pin *numbers* that were signal names instead of the
footprint's pad identifiers, so "Update PCB from Schematic" failed with
"pad not found" errors.

- J1 (USB4110-GF-A): shield pin number S1 -> SH to match the four "SH"
  shield pads in Connector_USB:USB_C_Receptacle_GCT_USB4110.
- U3 (MAX17048, DFN-8-1EP): renumber pins to the datasheet TDFN pads
  (CELL=2, GND=4, ALRT=5, QSTRT=6, SCL=7, SDA=8) and add the previously
  missing VDD (3), CTG (1) and exposed pad (9). VDD is stacked on the CELL
  node (VBAT, decoupled by C8) and CTG/EP on GND, so the gauge is actually
  powered - the prior symbol left VDD/CTG/EP unconnected.

Co-Authored-By: Claude Opus 4.8 <noreply@anthropic.com>
Claude-Session: https://claude.ai/code/session_019TySzotXwMtpz6QGTRfF9s
Connections:
- net ALRT: now also U3.5 (ALRT); no longer U3.ALRT
- net GND: now also U3.1 (CTG), U3.4 (GND), U3.6 (QSTRT), U3.9 (EP); no longer U3.GND, U3.QSTRT
- net SCL: now also U3.7 (SCL); no longer U3.SCL
- net SDA: now also U3.8 (SDA); no longer U3.SDA
- net VBAT: now also U3.2 (CELL), U3.3 (VDD); no longer U3.CELL
Changed lines of the file:
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@@
 		(property "Datasheet" "https://www.analog.com/media/en/technical-documentation/data-sheets/MAX17048-MAX17049.pdf" (at 90.00 55.00 0)
 			(effects (font (size 1.27 1.27)) (hide yes)))
-		(pin "CELL")
-		(pin "GND")
-		(pin "SDA")
-		(pin "SCL")
-		(pin "ALRT")
-		(pin "QSTRT")
+		(pin "2")
+		(pin "4")
+		(pin "8")
+		(pin "7")
+		(pin "5")
+		(pin "6")
+		(pin "3")
+		(pin "1")
+		(pin "9")
 		(instances
 			(project "cm4-carrier"
