File: hardware/cm4-carrier/cameras.kicad_sch (KiCad schematic)
At the start: 13 parts, among them J5 CSI Camera 0, J6 CSI Camera 1, U5 PCA9544APW, U7 AP2112K-3.3

Commit message: Add a DSI display on the CM4's DSI0 interface
Add a Raspberry Pi DSI display connector (J7) to the peripherals sheet
(now "Cameras & Display"):

- J7 is a standard 15-pin 1.0mm RPi FFC driven by the CM4's DSI0 (2-lane)
  interface; the six DSI0 differential lanes are exported from the CM4 sheet
  (J4) as global nets alongside the camera lanes.
- The display's touch/controller I2C shares I2C0 on PCA9544A mux channel 2
  (SD2/SC2, previously unused), with its own pull-ups (R21/R22).
- IO0/IO1 (reset / backlight-enable) route to CM4 GPIO8/GPIO9; 3.3V logic
  comes from the existing camera LDO rail. The 5V panel/backlight power is
  supplied separately, as on the standard RPi 7-inch panel.

The mux is now 3 of 4 channels used (cam0/cam1/display). Root box renamed to
"Cameras & Display". README/BOM updated. No format change (KiCad 10, 20260306).

Co-Authored-By: Claude Opus 4.8 <noreply@anthropic.com>
Claude-Session: https://claude.ai/code/session_015B7X7FE461jFSRaiTFdnFt
Parts:
- added J7: DSI Display 0, Connector_FFC-FPC:JUSHUO_AFA07-S15FCA-00_1x15-1MP_P1.0mm_Horizontal, symbol carrier:Raspberry_Pi_Camera_CSI
- added R21, R22: 4.7k, Resistor_SMD:R_0402_1005Metric, symbol carrier:R
Connections:
- net +3V3_CAM: now also J7.15 (VCC), R21.2, R22.2
- net GND: now also J7.1 (GND), J7.10 (GND), J7.4 (GND), J7.7 (GND)
- net DSI0_SDA: now reaches U5.12 (SD2)
- net DSI0_SDA: now also J7.14 (SDA), R21.1
- net DSI0_SCL: now reaches U5.13 (SC2)
- net DSI0_SCL: now also J7.13 (SCL), R22.1
- new net DSI0_C_N: J7.8 (CK_N)
- new net DSI0_C_P: J7.9 (CK_P)
- new net DSI0_D0_N: J7.2 (D0_N)
- new net DSI0_D0_P: J7.3 (D0_P)
- new net DSI0_D1_N: J7.5 (D1_N)
- new net DSI0_D1_P: J7.6 (D1_P)
- new net DSI0_IO0: J7.11 (IO0)
- new net DSI0_IO1: J7.12 (IO1)
- no-connect marks 10 -> 8
Other:
- note added: "CAM0->J5, CAM1->J6, DSI0 display->J7 (15-pin RPi FFCs). Local 3.3V LDO"
- note added: "Cameras & display - two CSI-2 cameras + one DSI display via a PCA9544A mux"
- note added: "powers them; the I2C mux (ch0/1/2) lets the same-address devices share I2C0."
- note removed: "CAM0 (2-lane) -> J5, CAM1 (4-lane, 2 used) -> J6. Local 3.3V LDO powers"
- note removed: "Dual CSI-2 cameras - two 15-pin RPi camera FFCs behind a PCA9544A mux"
- note removed: "the cameras; the I2C mux lets both same-address sensors share I2C0."

Commit message: hardware: vertical FFC + side-angle buttons/LEDs, all with 3D models
Swap three component families to right-angle / edge-mount parts that are
Digi-Key-stocked and map to KiCad footprints that ship with 3D models:

- FFC J5/J6/J7: horizontal JUSHUO/Amphenol -> TE 1-84982-5, 15-pos 1.0 mm
  *vertical* SMT socket (Connector_FFC-FPC:TE_1-84982-5_2Rows-15Pins-P1.0mm_Vertical).
- Tact switches SW1-SW6: SW_PUSH_6mm -> C&K PTS645VL39-2 LFS, 6 mm
  side-actuated right-angle THT (Button_Switch_THT:SW_Tactile_SPST_Angled_PTS645Vx39-2LFS).
- LEDs D1-D4: 0603 -> Kingbright APA1606 side-view / right-angle
  (LED_SMD:LED_Kingbright_APA1606_1.6x0.6mm_Horizontal).

All replacement footprints keep pad names compatible with their symbols
(FFC 1-15, switch/LED 1-2), so Update PCB from Schematic stays clean.

Audited every footprint in the design: all resolve to KiCad library
footprints with a 3D model (only the MountingHole pads have no body, as
expected). README BOM, sourcing notes and bom-digikey.csv updated with the
new manufacturer part numbers.

Co-Authored-By: Claude Opus 4.8 <noreply@anthropic.com>
Claude-Session: https://claude.ai/code/session_019TySzotXwMtpz6QGTRfF9s
Parts:
- J5, J6, J7: footprint Connector_FFC-FPC:JUSHUO_AFA07-S15FCA-00_1x15-1MP_P1.0mm_Horizontal -> Connector_FFC-FPC:TE_1-84982-5_2Rows-15Pins-P1.0mm_Vertical
Changed lines of the file:
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@@
 		(property "Value" "CSI Camera 0" (at 185.00 76.51 0)
 			(effects (font (size 1.27 1.27)) (justify left)))
-		(property "Footprint" "Connector_FFC-FPC:JUSHUO_AFA07-S15FCA-00_1x15-1MP_P1.0mm_Horizontal" (at 185.00 60.00 90)
+		(property "Footprint" "Connector_FFC-FPC:TE_1-84982-5_2Rows-15Pins-P1.0mm_Vertical" (at 185.00 60.00 90)
 			(effects (font (size 1.27 1.27)) (hide yes)))
 		(property "Datasheet" "" (at 185.00 60.00 0)
@@
 		(property "Value" "CSI Camera 1" (at 185.00 136.51 0)
 			(effects (font (size 1.27 1.27)) (justify left)))
-		(property "Footprint" "Connector_FFC-FPC:JUSHUO_AFA07-S15FCA-00_1x15-1MP_P1.0mm_Horizontal" (at 185.00 120.00 90)
+		(property "Footprint" "Connector_FFC-FPC:TE_1-84982-5_2Rows-15Pins-P1.0mm_Vertical" (at 185.00 120.00 90)
 			(effects (font (size 1.27 1.27)) (hide yes)))
 		(property "Datasheet" "" (at 185.00 120.00 0)
@@
 		(property "Value" "DSI Display 0" (at 185.00 196.51 0)
 			(effects (font (size 1.27 1.27)) (justify left)))
-		(property "Footprint" "Connector_FFC-FPC:JUSHUO_AFA07-S15FCA-00_1x15-1MP_P1.0mm_Horizontal" (at 185.00 180.00 90)
+		(property "Footprint" "Connector_FFC-FPC:TE_1-84982-5_2Rows-15Pins-P1.0mm_Vertical" (at 185.00 180.00 90)
 			(effects (font (size 1.27 1.27)) (hide yes)))
 		(property "Datasheet" "" (at 185.00 180.00 0)
