File: hardware/cm4-carrier/cameras.kicad_sch (KiCad schematic)
At the start: 16 parts, among them J5 CSI Camera 0, J6 CSI Camera 1, J7 DSI Display 0, U5 PCA9544APW, U7 AP2112K-3.3

Commit message: Revert "hardware: vertical FFC + side-angle buttons/LEDs, all with 3D models"
This reverts commit 6a117af7a4efdaa41e1a28fd110e1e5be4a57f55.
Parts:
- J5, J6, J7: footprint Connector_FFC-FPC:TE_1-84982-5_2Rows-15Pins-P1.0mm_Vertical -> Connector_FFC-FPC:JUSHUO_AFA07-S15FCA-00_1x15-1MP_P1.0mm_Horizontal
Changed lines of the file:
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@@
 		(property "Value" "CSI Camera 0" (at 185.00 76.51 0)
 			(effects (font (size 1.27 1.27)) (justify left)))
-		(property "Footprint" "Connector_FFC-FPC:TE_1-84982-5_2Rows-15Pins-P1.0mm_Vertical" (at 185.00 60.00 90)
+		(property "Footprint" "Connector_FFC-FPC:JUSHUO_AFA07-S15FCA-00_1x15-1MP_P1.0mm_Horizontal" (at 185.00 60.00 90)
 			(effects (font (size 1.27 1.27)) (hide yes)))
 		(property "Datasheet" "" (at 185.00 60.00 0)
@@
 		(property "Value" "CSI Camera 1" (at 185.00 136.51 0)
 			(effects (font (size 1.27 1.27)) (justify left)))
-		(property "Footprint" "Connector_FFC-FPC:TE_1-84982-5_2Rows-15Pins-P1.0mm_Vertical" (at 185.00 120.00 90)
+		(property "Footprint" "Connector_FFC-FPC:JUSHUO_AFA07-S15FCA-00_1x15-1MP_P1.0mm_Horizontal" (at 185.00 120.00 90)
 			(effects (font (size 1.27 1.27)) (hide yes)))
 		(property "Datasheet" "" (at 185.00 120.00 0)
@@
 		(property "Value" "DSI Display 0" (at 185.00 196.51 0)
 			(effects (font (size 1.27 1.27)) (justify left)))
-		(property "Footprint" "Connector_FFC-FPC:TE_1-84982-5_2Rows-15Pins-P1.0mm_Vertical" (at 185.00 180.00 90)
+		(property "Footprint" "Connector_FFC-FPC:JUSHUO_AFA07-S15FCA-00_1x15-1MP_P1.0mm_Horizontal" (at 185.00 180.00 90)
 			(effects (font (size 1.27 1.27)) (hide yes)))
 		(property "Datasheet" "" (at 185.00 180.00 0)
