File: hardware/cm4-carrier/power_input.kicad_sch (KiCad schematic)
At the start: 16 parts, among them J1 USB4110-GF-A, U1 BQ24075RGT

Commit message: Fix four footprint identifiers not found in KiCad libraries
"Update PCB from Schematic" reported four footprints missing; correct them to
the actual names in the current KiCad libraries (edited in place to preserve
symbol UUIDs, so existing PCB associations are kept):

- J1 USB-C: USB_C_Receptacle_GCT_USB4110-GF-A_16P_TopMnt_Horizontal
            -> USB_C_Receptacle_GCT_USB4110
- L1 inductor: L_Bourns-SRP1265A -> L_Bourns_SRP1245A (SRP1265A not in KiCad;
  pick the footprint matching your actual boost inductor)
- U1 BQ24075: VQFN-16-1EP_3x3mm_P0.5mm_EP1.7x1.7mm
            -> QFN-16-1EP_3x3mm_P0.5mm_EP1.7x1.7mm
- U3 MAX17048: DFN-8-1EP_2x2mm_P0.5mm_EP0.61x1.42mm
            -> DFN-8-1EP_2x2mm_P0.5mm_EP0.9x1.5mm

README BOM updated to match.

Co-Authored-By: Claude Opus 4.8 <noreply@anthropic.com>
Claude-Session: https://claude.ai/code/session_015B7X7FE461jFSRaiTFdnFt
Parts:
- J1: footprint Connector_USB:USB_C_Receptacle_GCT_USB4110-GF-A_16P_TopMnt_Horizontal -> Connector_USB:USB_C_Receptacle_GCT_USB4110
- U1: footprint Package_DFN_QFN:VQFN-16-1EP_3x3mm_P0.5mm_EP1.7x1.7mm -> Package_DFN_QFN:QFN-16-1EP_3x3mm_P0.5mm_EP1.7x1.7mm
Changed lines of the file:
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@@
 		(property "Value" "USB4110-GF-A" (at 45.00 66.43 0)
 			(effects (font (size 1.27 1.27)) (justify left)))
-		(property "Footprint" "Connector_USB:USB_C_Receptacle_GCT_USB4110-GF-A_16P_TopMnt_Horizontal" (at 45.00 55.00 90)
+		(property "Footprint" "Connector_USB:USB_C_Receptacle_GCT_USB4110" (at 45.00 55.00 90)
 			(effects (font (size 1.27 1.27)) (hide yes)))
 		(property "Datasheet" "https://gct.co/files/drawings/usb4110.pdf" (at 45.00 55.00 0)
@@
 		(property "Value" "BQ24075RGT" (at 115.00 87.24 0)
 			(effects (font (size 1.27 1.27)) (justify left)))
-		(property "Footprint" "Package_DFN_QFN:VQFN-16-1EP_3x3mm_P0.5mm_EP1.7x1.7mm" (at 115.00 72.00 90)
+		(property "Footprint" "Package_DFN_QFN:QFN-16-1EP_3x3mm_P0.5mm_EP1.7x1.7mm" (at 115.00 72.00 90)
 			(effects (font (size 1.27 1.27)) (hide yes)))
 		(property "Datasheet" "https://www.ti.com/lit/ds/symlink/bq24075.pdf" (at 115.00 72.00 0)

Commit message: hardware: fix J1/U3 symbol pad mapping for PCB update
Two custom symbols used pin *numbers* that were signal names instead of the
footprint's pad identifiers, so "Update PCB from Schematic" failed with
"pad not found" errors.

- J1 (USB4110-GF-A): shield pin number S1 -> SH to match the four "SH"
  shield pads in Connector_USB:USB_C_Receptacle_GCT_USB4110.
- U3 (MAX17048, DFN-8-1EP): renumber pins to the datasheet TDFN pads
  (CELL=2, GND=4, ALRT=5, QSTRT=6, SCL=7, SDA=8) and add the previously
  missing VDD (3), CTG (1) and exposed pad (9). VDD is stacked on the CELL
  node (VBAT, decoupled by C8) and CTG/EP on GND, so the gauge is actually
  powered - the prior symbol left VDD/CTG/EP unconnected.

Co-Authored-By: Claude Opus 4.8 <noreply@anthropic.com>
Claude-Session: https://claude.ai/code/session_019TySzotXwMtpz6QGTRfF9s
Connections:
- net GND: now also J1.SH (SHIELD); no longer J1.S1 (SHIELD)
Changed lines of the file:
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@@
 		(pin "A1")
 		(pin "A12")
-		(pin "S1")
+		(pin "SH")
 		(instances
 			(project "cm4-carrier"

Commit message: hardware: vertical FFC + side-angle buttons/LEDs, all with 3D models
Swap three component families to right-angle / edge-mount parts that are
Digi-Key-stocked and map to KiCad footprints that ship with 3D models:

- FFC J5/J6/J7: horizontal JUSHUO/Amphenol -> TE 1-84982-5, 15-pos 1.0 mm
  *vertical* SMT socket (Connector_FFC-FPC:TE_1-84982-5_2Rows-15Pins-P1.0mm_Vertical).
- Tact switches SW1-SW6: SW_PUSH_6mm -> C&K PTS645VL39-2 LFS, 6 mm
  side-actuated right-angle THT (Button_Switch_THT:SW_Tactile_SPST_Angled_PTS645Vx39-2LFS).
- LEDs D1-D4: 0603 -> Kingbright APA1606 side-view / right-angle
  (LED_SMD:LED_Kingbright_APA1606_1.6x0.6mm_Horizontal).

All replacement footprints keep pad names compatible with their symbols
(FFC 1-15, switch/LED 1-2), so Update PCB from Schematic stays clean.

Audited every footprint in the design: all resolve to KiCad library
footprints with a 3D model (only the MountingHole pads have no body, as
expected). README BOM, sourcing notes and bom-digikey.csv updated with the
new manufacturer part numbers.

Co-Authored-By: Claude Opus 4.8 <noreply@anthropic.com>
Claude-Session: https://claude.ai/code/session_019TySzotXwMtpz6QGTRfF9s
Parts:
- D1, D2: footprint LED_SMD:LED_0603_1608Metric -> LED_SMD:LED_Kingbright_APA1606_1.6x0.6mm_Horizontal
Changed lines of the file:
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@@
 		(property "Value" "CHG" (at 150.00 65.08 0)
 			(effects (font (size 1.27 1.27)) (justify left)))
-		(property "Footprint" "LED_SMD:LED_0603_1608Metric" (at 150.00 60.00 90)
+		(property "Footprint" "LED_SMD:LED_Kingbright_APA1606_1.6x0.6mm_Horizontal" (at 150.00 60.00 90)
 			(effects (font (size 1.27 1.27)) (hide yes)))
 		(property "Datasheet" "" (at 150.00 60.00 0)
@@
 		(property "Value" "PGOOD" (at 150.00 77.08 0)
 			(effects (font (size 1.27 1.27)) (justify left)))
-		(property "Footprint" "LED_SMD:LED_0603_1608Metric" (at 150.00 72.00 90)
+		(property "Footprint" "LED_SMD:LED_Kingbright_APA1606_1.6x0.6mm_Horizontal" (at 150.00 72.00 90)
 			(effects (font (size 1.27 1.27)) (hide yes)))
 		(property "Datasheet" "" (at 150.00 72.00 0)
