File: hardware/cm4-carrier/power_input.kicad_sch (KiCad schematic)
At the start: 16 parts, among them J1 USB4110-GF-A, U1 BQ24075RGT

Commit message: Revert "hardware: vertical FFC + side-angle buttons/LEDs, all with 3D models"
This reverts commit 6a117af7a4efdaa41e1a28fd110e1e5be4a57f55.
Parts:
- D1, D2: footprint LED_SMD:LED_Kingbright_APA1606_1.6x0.6mm_Horizontal -> LED_SMD:LED_0603_1608Metric
Changed lines of the file:
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@@
 		(property "Value" "CHG" (at 150.00 65.08 0)
 			(effects (font (size 1.27 1.27)) (justify left)))
-		(property "Footprint" "LED_SMD:LED_Kingbright_APA1606_1.6x0.6mm_Horizontal" (at 150.00 60.00 90)
+		(property "Footprint" "LED_SMD:LED_0603_1608Metric" (at 150.00 60.00 90)
 			(effects (font (size 1.27 1.27)) (hide yes)))
 		(property "Datasheet" "" (at 150.00 60.00 0)
@@
 		(property "Value" "PGOOD" (at 150.00 77.08 0)
 			(effects (font (size 1.27 1.27)) (justify left)))
-		(property "Footprint" "LED_SMD:LED_Kingbright_APA1606_1.6x0.6mm_Horizontal" (at 150.00 72.00 90)
+		(property "Footprint" "LED_SMD:LED_0603_1608Metric" (at 150.00 72.00 90)
 			(effects (font (size 1.27 1.27)) (hide yes)))
 		(property "Datasheet" "" (at 150.00 72.00 0)
