File: hardware/cm4-carrier/boot_sd.kicad_sch (KiCad schematic)
At the start: 32 parts, among them J8 microSD (CM4 Lite boot), Q2 DMG2305UX, Q3 2N7002, SW1 GLOBAL_EN, SW2 RUN_PG, SW3 nRPIBOOT, SW4 VOL_UP, SW5 VOL_DN, SW6 SLEEP/WAKE

Commit message: Revert "hardware: vertical FFC + side-angle buttons/LEDs, all with 3D models"
This reverts commit 6a117af7a4efdaa41e1a28fd110e1e5be4a57f55.
Parts:
- D3, D4: footprint LED_SMD:LED_Kingbright_APA1606_1.6x0.6mm_Horizontal -> LED_SMD:LED_0603_1608Metric
- SW1, SW2, SW3, SW4, SW5, SW6: footprint Button_Switch_THT:SW_Tactile_SPST_Angled_PTS645Vx39-2LFS -> Button_Switch_THT:SW_PUSH_6mm
Changed lines of the file:
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@@
 		(property "Value" "GLOBAL_EN" (at 72.00 150.08 0)
 			(effects (font (size 1.27 1.27)) (justify left)))
-		(property "Footprint" "Button_Switch_THT:SW_Tactile_SPST_Angled_PTS645Vx39-2LFS" (at 72.00 145.00 90)
+		(property "Footprint" "Button_Switch_THT:SW_PUSH_6mm" (at 72.00 145.00 90)
 			(effects (font (size 1.27 1.27)) (hide yes)))
 		(property "Datasheet" "" (at 72.00 145.00 0)
@@
 		(property "Value" "RUN_PG" (at 72.00 165.08 0)
 			(effects (font (size 1.27 1.27)) (justify left)))
-		(property "Footprint" "Button_Switch_THT:SW_Tactile_SPST_Angled_PTS645Vx39-2LFS" (at 72.00 160.00 90)
+		(property "Footprint" "Button_Switch_THT:SW_PUSH_6mm" (at 72.00 160.00 90)
 			(effects (font (size 1.27 1.27)) (hide yes)))
 		(property "Datasheet" "" (at 72.00 160.00 0)
@@
 		(property "Value" "nRPIBOOT" (at 72.00 180.08 0)
 			(effects (font (size 1.27 1.27)) (justify left)))
-		(property "Footprint" "Button_Switch_THT:SW_Tactile_SPST_Angled_PTS645Vx39-2LFS" (at 72.00 175.00 90)
+		(property "Footprint" "Button_Switch_THT:SW_PUSH_6mm" (at 72.00 175.00 90)
 			(effects (font (size 1.27 1.27)) (hide yes)))
 		(property "Datasheet" "" (at 72.00 175.00 0)
@@
 		(property "Value" "PWR" (at 120.00 155.08 0)
 			(effects (font (size 1.27 1.27)) (justify left)))
-		(property "Footprint" "LED_SMD:LED_Kingbright_APA1606_1.6x0.6mm_Horizontal" (at 120.00 150.00 90)
+		(property "Footprint" "LED_SMD:LED_0603_1608Metric" (at 120.00 150.00 90)
 			(effects (font (size 1.27 1.27)) (hide yes)))
 		(property "Datasheet" "" (at 120.00 150.00 0)
@@
 		(property "Value" "ACT" (at 120.00 170.08 0)
 			(effects (font (size 1.27 1.27)) (justify left)))
-		(property "Footprint" "LED_SMD:LED_Kingbright_APA1606_1.6x0.6mm_Horizontal" (at 120.00 165.00 90)
+		(property "Footprint" "LED_SMD:LED_0603_1608Metric" (at 120.00 165.00 90)
 			(effects (font (size 1.27 1.27)) (hide yes)))
 		(property "Datasheet" "" (at 120.00 165.00 0)
@@
 		(property "Value" "VOL_UP" (at 125.00 215.08 0)
 			(effects (font (size 1.27 1.27)) (justify left)))
-		(property "Footprint" "Button_Switch_THT:SW_Tactile_SPST_Angled_PTS645Vx39-2LFS" (at 125.00 210.00 90)
+		(property "Footprint" "Button_Switch_THT:SW_PUSH_6mm" (at 125.00 210.00 90)
 			(effects (font (size 1.27 1.27)) (hide yes)))
 		(property "Datasheet" "" (at 125.00 210.00 0)
@@
 		(property "Value" "VOL_DN" (at 125.00 230.08 0)
 			(effects (font (size 1.27 1.27)) (justify left)))
-		(property "Footprint" "Button_Switch_THT:SW_Tactile_SPST_Angled_PTS645Vx39-2LFS" (at 125.00 225.00 90)
+		(property "Footprint" "Button_Switch_THT:SW_PUSH_6mm" (at 125.00 225.00 90)
 			(effects (font (size 1.27 1.27)) (hide yes)))
 		(property "Datasheet" "" (at 125.00 225.00 0)
@@
 		(property "Value" "SLEEP/WAKE" (at 125.00 250.08 0)
 			(effects (font (size 1.27 1.27)) (justify left)))
-		(property "Footprint" "Button_Switch_THT:SW_Tactile_SPST_Angled_PTS645Vx39-2LFS" (at 125.00 245.00 90)
+		(property "Footprint" "Button_Switch_THT:SW_PUSH_6mm" (at 125.00 245.00 90)
 			(effects (font (size 1.27 1.27)) (hide yes)))
 		(property "Datasheet" "" (at 125.00 245.00 0)
